File: PCB_SCH/Geiger_EDW.kicad_pcb (KiCad board)
At the start: 2 copper layers, 120.1 x 46 mm, 48 parts, among them J1 Power, J2 +5V Output, J3 STS-5, J4 Piezo, J5 Output, P1 500k, Q1 IRF7404, Q2 BC857, Q3 IRFBC40SPBF, Q4 BC847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

Commit message: Update PCB values
Parts:
- R11: value 10k -> 1k
Changed lines of the file:
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@@
         (effects (font (size 1.016 1.016) (thickness 0.1524)))
     )
-    (fp_text value "10k" (at 0 1.82 90) (layer "F.Fab")
+    (fp_text value "1k" (at 0 1.82 90) (layer "F.Fab")
         (effects (font (size 1.016 1.016) (thickness 0.1524)))
     )
