File: PCB_SCH/Geiger_EDW.kicad_pcb (KiCad board)
At the start: 2 copper layers, 120.1 x 46 mm, 48 parts, among them J1 Power, J2 +5V Output, J3 STS-5, J4 Piezo, J5 Output, P1 500k, Q1 IRF7404, Q2 BC857, Q3 IRFBC40SPBF, Q4 BC847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

Commit message: Update components
Parts:
- added C12: 15p, Capacitor_THT:C_Disc_D3.0mm_W1.6mm_P2.50mm, F.Cu at (69.6, 129.5)
- added C13: 15p, Capacitor_THT:C_Disc_D3.0mm_W1.6mm_P2.50mm, F.Cu at (69.6, 132.7)
- added C14: 100n, Capacitor_THT:C_Disc_D3.8mm_W2.6mm_P2.50mm, F.Cu at (63.7, 118.2)
- added C15: 1n, Capacitor_THT:C_Disc_D3.8mm_W2.6mm_P2.50mm, F.Cu at (63.7, 122.3)
- added J6: Conn_01x03, Connector_PinHeader_2.54mm:PinHeader_1x03_P2.54mm_Vertical, F.Cu at (59.8, 118.4)
- added J7: Conn_01x14, Connector_PinHeader_2.54mm:PinHeader_1x14_P2.54mm_Vertical, F.Cu at (55.1, 100.1)
- added JP1: SolderJumper_3_Open, Jumper:SolderJumper-3_P2.0mm_Open_TrianglePad1.0x1.5mm_NumberLabels, F.Cu at (65.6, 126.2)
- added R1: 10k, Resistor_SMD:R_1206_3216Metric_Pad1.30x1.75mm_HandSolder, F.Cu at (65.1, 129.6)
- added R12: 330, Resistor_SMD:R_1206_3216Metric_Pad1.30x1.75mm_HandSolder, F.Cu at (65.1, 132.9)
- added RV1: 10k, Potentiometer_THT:Potentiometer_ACP_CA6-H2,5_Horizontal, F.Cu at (69.4, 117.7)
- added U4: ATmega8L-8A, Package_QFP:TQFP-32_7x7mm_P0.8mm, F.Cu at (63.3, 110.3)
- added Y1: 8MHz, Crystal:Crystal_HC18-U_Vertical, F.Cu at (61.5, 101.1)
- Q1: value IRF7404 -> AO4411
- Q3: value IRFBC40SPBF -> IXFA8N85XHV
