File: PCB_SCH/Geiger_EDW.kicad_sch (KiCad schematic)
At the start: 44 parts, among them J1 Power, J2 +5V Output, J3 STS-5, J4 Piezo, J5 Output, P1 500k, Q1 IRF7404, Q2 BC857, Q3 IRFBC40SPBF, Q4 BC847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

Commit message: New sheet, mcu added
Other:
- added sheet MCU_display (mcu_display.kicad_sch)
Changed lines of the file:
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@@
+    )
+  )
+  (sheet (at 300.99 0) (size 368.3 209.55) (fields_autoplaced)
+    (stroke (width 0.1524) (type solid))
+    (fill (color 0 0 0 0.0000))
+    (property "Sheetname" "MCU_display" (at 300.99 -0.7116 0)
+      (effects (font (size 1.27 1.27)) (justify left bottom))
+    )
+    (property "Sheetfile" "mcu_display.kicad_sch" (at 300.99 210.1346 0)
+      (effects (font (size 1.27 1.27)) (justify left top))
+    )
+    (instances
+      (project "Geiger_EDW"
+        (path "/3b22128b-b553-4988-96f2-c5a274af9a0d" (page "2"))
+      )
     )
   )
