File: PCB_SCH/Geiger_EDW.kicad_sch (KiCad schematic)
At the start: 44 parts, among them J1 Power, J2 +5V Output, J3 STS-5, J4 Piezo, J5 Output, P1 500k, Q1 IRF7404, Q2 BC857, Q3 IRFBC40SPBF, Q4 BC847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

Commit message: Update components
Parts:
- Q1: value IRF7404 -> AO4411
- Q3: value IRFBC40SPBF -> IXFA8N85XHV
Changed lines of the file:
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@@
       (effects (font (size 1.27 1.27)) (justify left))
     )
-    (property "Value" "IRFBC40SPBF" (at 85.09 41.91 0)
+    (property "Value" "IXFA8N85XHV" (at 85.09 41.91 0)
       (effects (font (size 1.27 1.27)) (justify left))
     )
@@
       (effects (font (size 1.27 1.27) italic) (justify left) hide)
     )
-    (property "Datasheet" "https://www.st.com/resource/en/datasheet/stp40n60m2.pdf" (at 96.52 35.56 0)
+    (property "Datasheet" "" (at 96.52 35.56 0)
       (effects (font (size 1.27 1.27)) (justify left) hide)
     )
@@
       (effects (font (size 1.27 1.27)) (justify left))
     )
-    (property "Value" "IRF7404" (at 73.66 86.36 0)
+    (property "Value" "AO4411" (at 73.66 86.36 0)
       (effects (font (size 1.27 1.27)) (justify left))
     )
@@
       (effects (font (size 1.27 1.27) italic) (justify left) hide)
     )
-    (property "Datasheet" "http://www.infineon.com/dgdl/irf7404.pdf?fileId=5546d462533600a4015355fa2b5b1b9e" (at 67.31 87.63 90)
+    (property "Datasheet" "" (at 67.31 87.63 90)
       (effects (font (size 1.27 1.27)) (justify left) hide)
     )
