File: PCB_SCH/mcu_display.kicad_sch (KiCad schematic)
At the start: 9 parts, among them J6 Conn_01x03, J7 Conn_01x14, U4 ATmega8L-8A, Y1 8MHz

Commit message: added jumper enabling selection between analog and digital contrast adjustment
Parts:
- added C15: 1n, Capacitor_THT:C_Disc_D3.8mm_W2.6mm_P2.50mm, symbol Device:C
- added JP1: SolderJumper_3_Open, Jumper:SolderJumper-3_P2.0mm_Open_TrianglePad1.0x1.5mm_NumberLabels, symbol Jumper:SolderJumper_3_Open
- added R12: 330, Resistor_SMD:R_1206_3216Metric_Pad1.30x1.75mm_HandSolder, symbol Device:R
Connections:
- net GND: now also C15.2
- net VE: now also JP1.2 (C); no longer RV1.2
- net at U4.13 (PB1): now also R12.1
- new net VE_ANA: JP1.3 (B), RV1.2
- new net VE_DIG: C15.1, JP1.1 (A), R12.2
Changed lines of the file:
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@@
   (junction (at 43.18 83.82) (diameter 0) (color 0 0 0 0)
   )
+  (junction (at 146.05 76.2) (diameter 0) (color 0 0 0 0)
+  )
   (wire (pts (xy 54.61 78.74) (xy 55.88 78.74))
     (stroke (width 0) (type default))
@@
     (stroke (width 0) (type default))
   )
+  (wire (pts (xy 146.05 86.36) (xy 146.05 91.44))
+    (stroke (width 0) (type default))
+  )
   (wire (pts (xy 95.25 137.16) (xy 95.25 154.94))
     (stroke (width 0) (type default))
@@
     (stroke (width 0) (type default))
   )
+  (wire (pts (xy 110.49 76.2) (xy 133.35 76.2))
+    (stroke (width 0) (type default))
+  )
   (wire (pts (xy 110.49 91.44) (xy 125.73 91.44))
     (stroke (width 0) (type default))
@@
     (stroke (width 0) (type default))
   )
+  (wire (pts (xy 140.97 76.2) (xy 146.05 76.2))
+    (stroke (width 0) (type default))
+  )
   (wire (pts (xy 80.01 88.9) (xy 68.58 88.9))
     (stroke (width 0) (type default))
@@
     (stroke (width 0) (type default))
   )
-  (wire (pts (xy 173.99 30.48) (xy 173.99 38.1))
-    (stroke (width 0) (type default))
-  )
-  (wire (pts (xy 67.31 34.29) (xy 81.28 34.29))
+  (wire (pts (xy 173.99 30.48) (xy 173.99 44.45))
     (stroke (width 0) (type default))
   )
@@
     (stroke (width 0) (type default))
   )
+  (wire (pts (xy 157.48 48.26) (xy 168.91 48.26))
+    (stroke (width 0) (type default))
+  )
   (wire (pts (xy 55.88 78.74) (xy 80.01 78.74))
     (stroke (width 0) (type default))
@@
     (stroke (width 0) (type default))
   )
+  (wire (pts (xy 146.05 76.2) (xy 152.4 76.2))
+    (stroke (width 0) (type default))
+  )
   (wire (pts (xy 97.79 54.61) (xy 97.79 66.04))
     (stroke (width 0) (type default))
@@
     (stroke (width 0) (type default))
   )
+  (wire (pts (xy 179.07 48.26) (xy 189.23 48.26))
+    (stroke (width 0) (type default))
+  )
   (wire (pts (xy 110.49 109.22) (xy 125.73 109.22))
     (stroke (width 0) (type default))
@@
     (stroke (width 0) (type default))
   )
+  (wire (pts (xy 146.05 76.2) (xy 146.05 78.74))
+    (stroke (width 0) (type default))
+  )
   (wire (pts (xy 110.49 83.82) (xy 125.73 83.82))
     (stroke (width 0) (type default))
@@
     (stroke (width 0) (type default))
   )
+  (wire (pts (xy 67.31 34.29) (xy 78.74 34.29))
+    (stroke (width 0) (type default))
+  )
   (label "GM_IMP" (at 118.11 73.66 0) (fields_autoplaced)
     (effects (font (size 1.27 1.27)) (justify left bottom))
   )
+  (label "VE_DIG" (at 143.51 76.2 0) (fields_autoplaced)
+    (effects (font (size 1.27 1.27)) (justify left bottom))
+  )
+  (label "VE_DIG" (at 180.34 48.26 0) (fields_autoplaced)
+    (effects (font (size 1.27 1.27)) (justify left bottom))
+  )
   (label "MISO" (at 118.11 83.82 0) (fields_autoplaced)
     (effects (font (size 1.27 1.27)) (justify left bottom))
@@
   )
   (label "RS" (at 176.53 36.83 90) (fields_autoplaced)
+    (effects (font (size 1.27 1.27)) (justify left bottom))
+  )
+  (label "VE_ANA" (at 161.29 48.26 0) (fields_autoplaced)
     (effects (font (size 1.27 1.27)) (justify left bottom))
   )
@@
     (effects (font (size 1.27 1.27)) (justify left bottom))
   )
-  (label "VE" (at 69.85 34.29 0) (fields_autoplaced)
+  (label "VE_ANA" (at 69.85 34.29 0) (fields_autoplaced)
     (effects (font (size 1.27 1.27)) (justify left bottom))
   )
@@
     )
   )
+  (symbol (lib_id "Device:C") (at 146.05 82.55 0) (unit 1)
+    (in_bom yes) (on_board yes) (dnp no) (fields_autoplaced)
+    (property "Reference" "C15" (at 149.86 81.28 0)
+      (effects (font (size 1.27 1.27)) (justify left))
+    )
+    (property "Value" "1n" (at 149.86 83.82 0)
+      (effects (font (size 1.27 1.27)) (justify left))
+    )
+    (property "Footprint" "Capacitor_THT:C_Disc_D3.8mm_W2.6mm_P2.50mm" (at 147.0152 86.36 0)
+      (effects (font (size 1.27 1.27)) hide)
+    )
+    (property "Datasheet" "~" (at 146.05 82.55 0)
+      (effects (font (size 1.27 1.27)) hide)
+    )
+    (pin "1")
+    (pin "2")
+    (instances
+      (project "Geiger_EDW"
+        (path "/3b22128b-b553-4988-96f2-c5a274af9a0d/c4286dcc-ecc2-4be7-a89d-80887accf133"
+          (reference "C15") (unit 1)
+        )
+      )
+    )
+  )
   (symbol (lib_id "power:GND") (at 63.5 41.91 0) (unit 1)
     (in_bom yes) (on_board yes) (dnp no) (fields_autoplaced)
@@
     )
   )
+  (symbol (lib_id "Jumper:SolderJumper_3_Open") (at 173.99 48.26 180) (unit 1)
+    (in_bom yes) (on_board yes) (dnp no) (fields_autoplaced)
+    (property "Reference" "JP1" (at 173.99 52.07 0)
+      (effects (font (size 1.27 1.27)))
+    )
+    (property "Value" "SolderJumper_3_Open" (at 173.99 54.61 0)
+      (effects (font (size 1.27 1.27)))
+    )
+    (property "Footprint" "Jumper:SolderJumper-3_P2.0mm_Open_TrianglePad1.0x1.5mm_NumberLabels" (at 173.99 48.26 0)
+      (effects (font (size 1.27 1.27)) hide)
+    )
+    (property "Datasheet" "~" (at 173.99 48.26 0)
+      (effects (font (size 1.27 1.27)) hide)
+    )
+    (pin "1")
+    (pin "2")
+    (pin "3")
+    (instances
+      (project "Geiger_EDW"
+        (path "/3b22128b-b553-4988-96f2-c5a274af9a0d/c4286dcc-ecc2-4be7-a89d-80887accf133"
+          (reference "JP1") (unit 1)
+        )
+      )
+    )
+  )
   (symbol (lib_id "Device:R") (at 63.5 64.77 0) (unit 1)
     (in_bom yes) (on_board yes) (dnp no) (fields_autoplaced)
@@
         (path "/3b22128b-b553-4988-96f2-c5a274af9a0d/c4286dcc-ecc2-4be7-a89d-80887accf133"
           (reference "R1") (unit 1)
+        )
+      )
+    )
+  )
+  (symbol (lib_id "power:GND") (at 146.05 91.44 0) (unit 1)
+    (in_bom yes) (on_board yes) (dnp no) (fields_autoplaced)
+    (property "Reference" "#PWR026" (at 146.05 97.79 0)
+      (effects (font (size 1.27 1.27)) hide)
+    )
+    (property "Value" "GND" (at 146.05 96.52 0)
+      (effects (font (size 1.27 1.27)))
+    )
+    (property "Footprint" "" (at 146.05 91.44 0)
+      (effects (font (size 1.27 1.27)) hide)
+    )
+    (property "Datasheet" "" (at 146.05 91.44 0)
+      (effects (font (size 1.27 1.27)) hide)
+    )
+    (pin "1")
+    (instances
+      (project "Geiger_EDW"
+        (path "/3b22128b-b553-4988-96f2-c5a274af9a0d/c4286dcc-ecc2-4be7-a89d-80887accf133"
+          (reference "#PWR026") (unit 1)
         )
       )
@@
         )
       )
+    )
+  )
+  (symbol (lib_id "Device:R") (at 137.16 76.2 90) (unit 1)
+    (in_bom yes) (on_board yes) (dnp no) (fields_autoplaced)
+    (property "Reference" "R12" (at 137.16 69.85 90)
+      (effects (font (size 1.27 1.27)))
+    )
+    (property "Value" "330" (at 137.16 72.39 90)
+      (effects (font (size 1.27 1.27)))
+    )
+    (property "Footprint" "Resistor_SMD:R_1206_3216Metric_Pad1.30x1.75mm_HandSolder" (at 137.16 77.978 90)
+      (effects (font (size 1.27 1.27)) hide)
+    )
+    (property "Datasheet" "~" (at 137.16 76.2 0)
+      (effects (font (size 1.27 1.27)) hide)
+    )
+    (pin "1")
+    (pin "2")
+    (instances
+      (project "Geiger_EDW"
+        (path "/3b22128b-b553-4988-96f2-c5a274af9a0d/c4286dcc-ecc2-4be7-a89d-80887accf133"
+          (reference "R12") (unit 1)
+        )
+      )
